Commit message: arm attached to chassis

File: robot/description/robot_arm.xacro (robot description, xacro)
@@ -6,5 +6,5 @@
       <parent link="base_link"/>
       <child link="arm_base"/>
-      <origin rpy="0 0 0" xyz="0.0 0.0 0.18"/>
+      <origin rpy="0 0 0" xyz="0.0 0.0 0.15"/>
    </joint>
    <link name="arm_base">

Commit message: joint order redone

File: robot/description/robot_arm.xacro (robot description, xacro)
@@ -79,4 +79,82 @@
       <turnGravityOff>true</turnGravityOff>
    </gazebo>
+   <!-- BOTTON WRIST -->
+   <joint name="bottom_wrist_joint" type="continuous">
+      <axis xyz="0 1 0"/>
+      <parent link="bicep"/>
+      <child link="bottom_wrist"/>
+      <origin rpy="0 0 0" xyz="0.0 -0.05194 0.269"/>
+   </joint>
+   <link name="bottom_wrist">
+      <inertial>
+         <origin xyz="-9.1053E-08 -0.069257 -1.86629999995759E-07" rpy="0 0 0" />
+         <mass value="0.27721" />
+         <inertia
+            ixx="0.00104290750143942"
+            ixy="4.37155302268076E-09"
+            ixz="-2.45049603914627E-09"
+            iyy="0.000380518373895034"
+            iyz="-7.56009835172156E-09"
+            izz="0.00106006525067445" />
+      </inertial>
+      <visual>
+         <origin xyz="0 0 0.13522" rpy="3.14 0 1.5708" />
+         <geometry>
+            <mesh filename="file://$(find robot)/description/meshes/wrist.stl" />
+         </geometry>
+         <material name="">
+         <color rgba="0.79216 0.81961 0.93333 1" />
+      </material>
+    </visual>
+      <collision>
+         <origin xyz="0 0 0.13522" rpy="3.14 0 1.5708" />
+         <geometry>
+            <mesh filename="file://$(find robot)/description/meshes/wrist.stl" />
+         </geometry>
+      </collision>
+   </link>
+   <gazebo reference="bottom_wrist">
+      <material>Gazebo/White</material>
+      <turnGravityOff>true</turnGravityOff>
+   </gazebo>
+   <!-- ELBOW -->
+   <joint name="elbow_joint" type="continuous">
+      <axis xyz="0 0 1"/>
+      <parent link="bottom_wrist"/>
+      <child link="elbow"/>
+      <origin rpy="0 0 0" xyz="0.0 0 0.13522"/>
+   </joint>
+  <link name="elbow">
+      <inertial>
+         <origin xyz="-0.11109 1.1476E-08 0.046469" rpy="0 0 0" />
+         <mass value="0.84845" />
+         <inertia
+            ixx="0.00079656"
+            ixy="-7.8011E-10"
+            ixz="0.00053616"
+            iyy="0.003576"
+            iyz="4.6326E-10"
+            izz="0.0033698" />
+      </inertial>
+      <visual>
+         <origin xyz="0.0 0.05163 0.20994" rpy="0 -1.5708 0" />
+         <geometry>
+            <mesh filename="file://$(find robot)/description/meshes/elbow.stl" />
+         </geometry>
+         <material name="">
+            <color rgba="0.79216 0.81961 0.93333 1" />
+         </material>
+      </visual>
+      <collision>
+         <origin xyz="0.0 0.05163 0.20994" rpy="0 -1.5708 0" />
+         <geometry>
+            <mesh filename="file://$(find robot)/description/meshes/elbow.stl" />
+         </geometry>
+      </collision>
+   </link>
+   <gazebo reference="elbow">
+      <material>Gazebo/White</material>
+      <turnGravityOff>true</turnGravityOff>
+   </gazebo>
    <!-- TOP WRIST -->
    <joint name="top_wrist_joint" type="continuous">
@@ -118,82 +196,4 @@
       <turnGravityOff>true</turnGravityOff>
    </gazebo>
-   <!-- BOTTON WRIST -->
-   <joint name="bottom_wrist_joint" type="continuous">
-      <axis xyz="0 1 0"/>
-      <parent link="bicep"/>
-      <child link="bottom_wrist"/>
-      <origin rpy="0 0 0" xyz="0.0 -0.05194 0.269"/>
-   </joint>
-   <link name="bottom_wrist">
-      <inertial>
-         <origin xyz="-9.1053E-08 -0.069257 -1.86629999995759E-07" rpy="0 0 0" />
-         <mass value="0.27721" />
-         <inertia
-            ixx="0.00104290750143942"
-            ixy="4.37155302268076E-09"
-            ixz="-2.45049603914627E-09"
-            iyy="0.000380518373895034"
-            iyz="-7.56009835172156E-09"
-            izz="0.00106006525067445" />
-      </inertial>
-      <visual>
-         <origin xyz="0 0 0.13522" rpy="3.14 0 1.5708" />
-         <geometry>
-            <mesh filename="file://$(find robot)/description/meshes/wrist.stl" />
-         </geometry>
-         <material name="">
-         <color rgba="0.79216 0.81961 0.93333 1" />
-      </material>
-    </visual>
-      <collision>
-         <origin xyz="0 0 0.13522" rpy="3.14 0 1.5708" />
-         <geometry>
-            <mesh filename="file://$(find robot)/description/meshes/wrist.stl" />
-         </geometry>
-      </collision>
-   </link>
-   <gazebo reference="bottom_wrist">
-      <material>Gazebo/White</material>
-      <turnGravityOff>true</turnGravityOff>
-   </gazebo>
-   <!-- ELBOW -->
-   <joint name="elbow_joint" type="continuous">
-      <axis xyz="0 0 1"/>
-      <parent link="bottom_wrist"/>
-      <child link="elbow"/>
-      <origin rpy="0 0 0" xyz="0.0 0 0.13522"/>
-   </joint>
-  <link name="elbow">
-      <inertial>
-         <origin xyz="-0.11109 1.1476E-08 0.046469" rpy="0 0 0" />
-         <mass value="0.84845" />
-         <inertia
-            ixx="0.00079656"
-            ixy="-7.8011E-10"
-            ixz="0.00053616"
-            iyy="0.003576"
-            iyz="4.6326E-10"
-            izz="0.0033698" />
-      </inertial>
-      <visual>
-         <origin xyz="0.0 0.05163 0.20994" rpy="0 -1.5708 0" />
-         <geometry>
-            <mesh filename="file://$(find robot)/description/meshes/elbow.stl" />
-         </geometry>
-         <material name="">
-            <color rgba="0.79216 0.81961 0.93333 1" />
-         </material>
-      </visual>
-      <collision>
-         <origin xyz="0.0 0.05163 0.20994" rpy="0 -1.5708 0" />
-         <geometry>
-            <mesh filename="file://$(find robot)/description/meshes/elbow.stl" />
-         </geometry>
-      </collision>
-   </link>
-   <gazebo reference="elbow">
-      <material>Gazebo/White</material>
-      <turnGravityOff>true</turnGravityOff>
-   </gazebo>
    <!-- TRANSMISSIONS -->
   <transmission name="arm_base_trans" type="SimpleTransmission">
