Commit message: arm_almost_working

File: robot/description/gazebo_control.xacro (robot description, xacro)
@@ -26,7 +26,20 @@
         </plugin>
     </gazebo>
+    <!-- <gazebo>
+        <plugin name="gazebo_ros_joint_state_publisher"
+            filename="libgazebo_ros_joint_state_publisher.so">
+            <update_rate>20</update_rate>
+            <joint_name>slider_joint</joint_name>
+            <joint_name>arm_joint</joint_name>
+        </plugin>
+    </gazebo> -->
     <gazebo>
         <plugin name="joint_state_publisher" filename="libgazebo_ros_joint_state_publisher.so">
-            <jointName>arm_base_joint, shoulder_joint, bottom_wrist_joint, elbow_joint, top_wrist_joint</jointName>
+            <update_rate>20</update_rate>
+            <joint_name>arm_base_joint</joint_name>
+            <joint_name>shoulder_joint</joint_name>
+            <joint_name>bottom_wrist_joint</joint_name>
+            <joint_name>elbow_joint</joint_name>
+            <joint_name>top_wrist_joint</joint_name>
         </plugin>
     </gazebo>

File: robot/description/robot.urdf.xacro (robot description, xacro)
@@ -3,5 +3,5 @@
     <xacro:include filename="robot_core.xacro" />
     <xacro:include filename="gazebo_control.xacro" />
-    <xacro:include filename="gazebo_lidar.xacro" />
+    <!-- <xacro:include filename="gazebo_lidar.xacro" />  -->
     <xacro:include filename="robot_lidar.xacro" />
     <xacro:include filename="robot_arm.xacro" />

File: robot/description/robot_arm.xacro (robot description, xacro)
@@ -4,5 +4,5 @@
    <joint name="arm_base_joint" type="continuous">
       <axis xyz="0 0 1"/>
-      <parent link="chassis"/>
+      <parent link="base_link"/>
       <child link="arm_base"/>
       <origin rpy="0 0 0" xyz="0.0 0.0 0.18"/>
@@ -23,5 +23,5 @@
          <origin xyz="0 0 0" rpy="0 0 0" />
          <geometry>
-            <mesh filename="file://$(find robot)/description/meshes/arm_base.stl" />
+            <mesh filename="file://$(find robot)/description/meshes/arm_base.stl"/>
          </geometry>
          <material name="">
@@ -32,5 +32,5 @@
          <origin xyz="0 0 0" rpy="0 0 0" />
          <geometry>
-            <mesh filename="file://$(find robot)/description/meshes/arm_base.stl" />
+            <mesh filename="file://$(find robot)/description/meshes/arm_base.stl"/>
          </geometry>
       </collision>

File: robot/description/robot_core.xacro (robot description, xacro)
@@ -96,5 +96,5 @@
       <material>Gazebo/Blue</material>
    </gazebo>
-   <!-- CASTER WHEEL LINK -->
+   <!-- CASTER WHEEL FRONT -->
    <joint name="caster_wheel_joint" type="fixed">
       <parent link="chassis" />
@@ -123,3 +123,30 @@
       <mu2 value="0.001" />
    </gazebo>
+   <!-- CASTER WHEEL BACK -->
+   <joint name="back_caster_wheel_joint" type="fixed">
+      <parent link="chassis" />
+      <child link="back_caster_wheel" />
+      <origin xyz="0.05 0 0" />
+   </joint>
+   <link name="back_caster_wheel">
+      <visual>
+         <geometry>
+            <sphere radius="0.05" />
+         </geometry>
+         <material name="black" />
+      </visual>
+      <collision>
+         <geometry>
+            <sphere radius="0.05" />
+         </geometry>
+      </collision>
+      <xacro:inertial_sphere mass="0.1" radius="0.05">
+         <origin xyz="0 0 0" rpy="0 0 0" />
+      </xacro:inertial_sphere>
+   </link>
+   <gazebo reference="back_caster_wheel">
+      <material>Gazebo/Black</material>
+      <mu1 value="0.001" />
+      <mu2 value="0.001" />
+   </gazebo>
 </robot>

Commit message: control_almost_working

File: robot/description/gazebo_control.xacro (robot description, xacro)
@@ -19,9 +19,30 @@
         </plugin>
     </gazebo>
-    <gazebo>
+    <ros2_control name="GazeboSystem" type="system">
+        <hardware>
+            <plugin>gazebo_ros2_control/GazeboSystem</plugin>
+        </hardware>
+        <joint name="arm_base_joint">
+            <command_interface name="position">
+                <param name="min">-1000</param>
+                <param name="max">1000</param>
+            </command_interface>
+            <state_interface name="position"/>
+            <state_interface name="velocity"/>
+            <state_interface name="effort"/>
+        </joint>
+    </ros2_control>
+    <!-- <gazebo>
         <plugin name="gazebo_ros_control" filename="libgazebo_ros_control.so">
-            <robotNamespace>/</robotNamespace>
+            <robotNamespace>/robot</robotNamespace>
             <controlPeriod>0.001</controlPeriod>
             <legacyModeNS>false</legacyModeNS>
+        </plugin>
+    </gazebo> -->
+    <gazebo>
+        <plugin filename="libgazebo_ros2_control.so" name="gazebo_ros2_control">
+            <robot_param>robot_description</robot_param>
+            <robot_param_node>robot_state_publisher</robot_param_node>
+            <parameters>$(find robot)/config/robot.yaml</parameters>
         </plugin>
     </gazebo>
@@ -34,5 +55,5 @@
         </plugin>
     </gazebo> -->
-    <gazebo>
+    <!-- <gazebo>
         <plugin name="joint_state_publisher" filename="libgazebo_ros_joint_state_publisher.so">
             <update_rate>20</update_rate>
@@ -43,4 +64,4 @@
             <joint_name>top_wrist_joint</joint_name>
         </plugin>
-    </gazebo>
+    </gazebo> -->
 </robot>

File: robot/description/robot_arm.xacro (robot description, xacro)
@@ -37,5 +37,5 @@
    </link>
    <!-- BICEP -->
-   <joint name="shoulder_joint" type="continuous">
+   <!-- <joint name="shoulder_joint" type="continuous">
       <axis xyz="0 1 0"/>
       <parent link="arm_base"/>
@@ -70,7 +70,7 @@
          </geometry>
       </collision>
-   </link>
+   </link> -->
    <!-- TOP WRIST -->
-   <joint name="top_wrist_joint" type="continuous">
+   <!-- <joint name="top_wrist_joint" type="continuous">
       <axis xyz="0 1 0"/>
       <parent link="elbow"/>
@@ -105,7 +105,7 @@
          </geometry>
       </collision>
-   </link>
+   </link> -->
    <!-- BOTTON WRIST -->
-   <joint name="bottom_wrist_joint" type="continuous">
+   <!-- <joint name="bottom_wrist_joint" type="continuous">
       <axis xyz="0 1 0"/>
       <parent link="bicep"/>
@@ -140,7 +140,7 @@
          </geometry>
       </collision>
-   </link>
+   </link> -->
    <!-- ELBOW -->
-   <joint name="elbow_joint" type="continuous">
+   <!-- <joint name="elbow_joint" type="continuous">
       <axis xyz="0 0 1"/>
       <parent link="bottom_wrist"/>
@@ -175,5 +175,5 @@
          </geometry>
       </collision>
-  </link>
+  </link> -->
    <!-- TRANSMISSIONS -->
   <transmission name="arm_base_trans" type="SimpleTransmission">
@@ -187,5 +187,5 @@
       </joint>
    </transmission>
-   <transmission name="shoulder_trans" type="SimpleTransmission">
+   <!-- <transmission name="shoulder_trans" type="SimpleTransmission">
       <type>transmission_interface/SimpleTransmission</type>
       <actuator name="shoulder_motor">
@@ -226,4 +226,4 @@
          <hardwareInterface>hardware_interface/PositionJointInterface</hardwareInterface>
       </joint>
-   </transmission>
+   </transmission> -->
 </robot>

Commit message: inertial_problems!

File: robot/description/gazebo_control.xacro (robot description, xacro)
@@ -25,6 +25,42 @@
         <joint name="arm_base_joint">
             <command_interface name="position">
-                <param name="min">-1000</param>
-                <param name="max">1000</param>
+                <param name="min">-1</param>
+                <param name="max">1</param>
+            </command_interface>
+            <state_interface name="position"/>
+            <state_interface name="velocity"/>
+            <state_interface name="effort"/>
+        </joint>
+        <joint name="shoulder_joint">
+            <command_interface name="position">
+                <param name="min">-1</param>
+                <param name="max">1</param>
+            </command_interface>
+            <state_interface name="position"/>
+            <state_interface name="velocity"/>
+            <state_interface name="effort"/>
+        </joint>
+        <joint name="top_wrist_joint">
+            <command_interface name="position">
+                <param name="min">-1</param>
+                <param name="max">1</param>
+            </command_interface>
+            <state_interface name="position"/>
+            <state_interface name="velocity"/>
+            <state_interface name="effort"/>
+        </joint>
+        <joint name="bottom_wrist_joint">
+            <command_interface name="position">
+                <param name="min">-1</param>
+                <param name="max">1</param>
+            </command_interface>
+            <state_interface name="position"/>
+            <state_interface name="velocity"/>
+            <state_interface name="effort"/>
+        </joint>
+        <joint name="elbow_joint">
+            <command_interface name="position">
+                <param name="min">-1</param>
+                <param name="max">1</param>
             </command_interface>
             <state_interface name="position"/>

File: robot/description/robot_arm.xacro (robot description, xacro)
@@ -36,6 +36,9 @@
       </collision>
    </link>
+   <gazebo reference="arm_base">
+      <material>Gazebo/White</material>
+   </gazebo>
    <!-- BICEP -->
-   <!-- <joint name="shoulder_joint" type="continuous">
+   <joint name="shoulder_joint" type="continuous">
       <axis xyz="0 1 0"/>
       <parent link="arm_base"/>
@@ -70,7 +73,10 @@
          </geometry>
       </collision>
-   </link> -->
+   </link>
+   <gazebo reference="bicep">
+      <material>Gazebo/White</material>
+   </gazebo>
    <!-- TOP WRIST -->
-   <!-- <joint name="top_wrist_joint" type="continuous">
+   <joint name="top_wrist_joint" type="continuous">
       <axis xyz="0 1 0"/>
       <parent link="elbow"/>
@@ -105,7 +111,10 @@
          </geometry>
       </collision>
-   </link> -->
+   </link>
+   <gazebo reference="top_wrist">
+      <material>Gazebo/White</material>
+   </gazebo>
    <!-- BOTTON WRIST -->
-   <!-- <joint name="bottom_wrist_joint" type="continuous">
+   <joint name="bottom_wrist_joint" type="continuous">
       <axis xyz="0 1 0"/>
       <parent link="bicep"/>
@@ -140,7 +149,10 @@
          </geometry>
       </collision>
-   </link> -->
+   </link>
+   <gazebo reference="bottom_wrist">
+      <material>Gazebo/White</material>
+   </gazebo>
    <!-- ELBOW -->
-   <!-- <joint name="elbow_joint" type="continuous">
+   <joint name="elbow_joint" type="continuous">
       <axis xyz="0 0 1"/>
       <parent link="bottom_wrist"/>
@@ -175,24 +187,27 @@
          </geometry>
       </collision>
-  </link> -->
+   </link>
+   <gazebo reference="elbow">
+      <material>Gazebo/White</material>
+   </gazebo>
    <!-- TRANSMISSIONS -->
   <transmission name="arm_base_trans" type="SimpleTransmission">
       <type>transmission_interface/SimpleTransmission</type>
       <actuator name="arm_base_motor">
-         <hardwareInterface>hardware_interface/PositionJointInterface</hardwareInterface>
+         <hardwareInterface>EffortJointInterface</hardwareInterface>
          <mechanicalReduction>1</mechanicalReduction>
       </actuator>
       <joint name="arm_base_joint">
-         <hardwareInterface>hardware_interface/PositionJointInterface</hardwareInterface>
-      </joint>
-   </transmission>
-   <!-- <transmission name="shoulder_trans" type="SimpleTransmission">
+         <hardwareInterface>EffortJointInterface</hardwareInterface>
+      </joint>
+   </transmission>
+   <transmission name="shoulder_trans" type="SimpleTransmission">
       <type>transmission_interface/SimpleTransmission</type>
       <actuator name="shoulder_motor">
-         <hardwareInterface>hardware_interface/PositionJointInterface</hardwareInterface>
+         <hardwareInterface>EffortJointInterface</hardwareInterface>
          <mechanicalReduction>1</mechanicalReduction>
       </actuator>
       <joint name="shoulder_joint">
-         <hardwareInterface>hardware_interface/PositionJointInterface</hardwareInterface>
+         <hardwareInterface>EffortJointInterface</hardwareInterface>
       </joint>
    </transmission>
@@ -200,9 +215,9 @@
       <type>transmission_interface/SimpleTransmission</type>
       <actuator name="bottom_wrist_motor">
-         <hardwareInterface>hardware_interface/PositionJointInterface</hardwareInterface>
+         <hardwareInterface>EffortJointInterface</hardwareInterface>
          <mechanicalReduction>1</mechanicalReduction>
       </actuator>
       <joint name="bottom_wrist_joint">
-         <hardwareInterface>hardware_interface/PositionJointInterface</hardwareInterface>
+         <hardwareInterface>EffortJointInterface</hardwareInterface>
       </joint>
    </transmission>
@@ -210,9 +225,9 @@
       <type>transmission_interface/SimpleTransmission</type>
       <actuator name="elbow_motor">
-         <hardwareInterface>hardware_interface/PositionJointInterface</hardwareInterface>
+         <hardwareInterface>EffortJointInterface</hardwareInterface>
          <mechanicalReduction>1</mechanicalReduction>
       </actuator>
       <joint name="elbow_joint">
-         <hardwareInterface>hardware_interface/PositionJointInterface</hardwareInterface>
+         <hardwareInterface>EffortJointInterface</hardwareInterface>
       </joint>
    </transmission>
@@ -220,10 +235,10 @@
       <type>transmission_interface/SimpleTransmission</type>
       <actuator name="top_wrist_motor">
-         <hardwareInterface>hardware_interface/PositionJointInterface</hardwareInterface>
+         <hardwareInterface>EffortJointInterface</hardwareInterface>
          <mechanicalReduction>1</mechanicalReduction>
       </actuator>
       <joint name="top_wrist_joint">
-         <hardwareInterface>hardware_interface/PositionJointInterface</hardwareInterface>
-      </joint>
-   </transmission> -->
+         <hardwareInterface>EffortJointInterface</hardwareInterface>
+      </joint>
+   </transmission>
 </robot>

Commit message: pinch

File: robot/description/gazebo_control.xacro (robot description, xacro)
@@ -68,4 +68,22 @@
             <state_interface name="effort"/>
         </joint>
+        <joint name="plier_right_joint">
+            <command_interface name="position">
+                <param name="min">-1</param>
+                <param name="max">1</param>
+            </command_interface>
+            <state_interface name="position"/>
+            <state_interface name="velocity"/>
+            <state_interface name="effort"/>
+        </joint>
+        <joint name="plier_left_joint">
+            <command_interface name="position">
+                <param name="min">-1</param>
+                <param name="max">1</param>
+            </command_interface>
+            <state_interface name="position"/>
+            <state_interface name="velocity"/>
+            <state_interface name="effort"/>
+        </joint>
     </ros2_control>
     <!-- <gazebo>

File: robot/description/robot_arm.xacro (robot description, xacro)
@@ -196,4 +196,98 @@
       <turnGravityOff>true</turnGravityOff>
    </gazebo>
+   <!-- PLIER BASE -->
+   <joint name="plier_base_joint" type="fixed">
+      <parent link="top_wrist"/>
+      <child link="plier_base"/>
+      <origin rpy="-${pi/2} -${pi/2} -${pi/2}" xyz="0 0 0.14"/>
+   </joint>
+   <link name="plier_base">
+      <visual>
+         <origin xyz="0 0 0" />
+         <geometry>
+            <box size="0.02 0.15 0.20" />
+         </geometry>
+         <material name="">
+            <color rgba="0.79216 0.81961 0.93333 1" />
+         </material>
+      </visual>
+      <collision>
+         <origin xyz="0 0 0" />
+         <geometry>
+            <box size="0.02 0.15 0.30" />
+         </geometry>
+      </collision>
+      <xacro:inertial_box mass="0.5" x="0.02" y="0.15" z="0.20">
+         <origin xyz="0 0 0" rpy="0 0 0" />
+      </xacro:inertial_box>
+   </link>
+   <gazebo reference="plier_base">
+      <material>Gazebo/White</material>
+      <turnGravityOff>true</turnGravityOff>
+   </gazebo>
+   <!-- PLIER RIGHT -->
+   <joint name="plier_right_joint" type="prismatic">
+      <limit effort="1000.0" lower="0" upper="0.2" velocity="0.5"/>
+      <axis xyz="1 0 0"/>
+      <parent link="plier_base"/>
+      <child link="plier_right"/>
+      <origin rpy="-${pi/2} -${pi/2} -${pi/2} " xyz="0.085 0 -0.088"/>
+   </joint>
+   <link name="plier_right">
+      <visual>
+         <origin xyz="0 0 0" />
+         <geometry>
+            <box size="0.02 0.15 0.15" />
+         </geometry>
+         <material name="">
+            <color rgba="0.79216 0.81961 0.93333 1" />
+         </material>
+      </visual>
+      <collision>
+         <origin xyz="0 0 0" />
+         <geometry>
+            <box size="0.02 0.15 0.15" />
+         </geometry>
+      </collision>
+      <xacro:inertial_box mass="0.5" x="0.02" y="0.15" z="0.15">
+         <origin xyz="0 0 0" rpy="0 0 0" />
+      </xacro:inertial_box>
+   </link>
+   <gazebo reference="plier_right">
+      <material>Gazebo/White</material>
+      <turnGravityOff>true</turnGravityOff>
+   </gazebo>
+   <!-- PLIER LEFT -->
+   <joint name="plier_left_joint" type="prismatic">
+      <limit effort="1000.0" lower="0" upper="0.2" velocity="0.5"/>
+      <axis xyz="-1 0 0"/>
+      <parent link="plier_base"/>
+      <child link="plier_left"/>
+      <origin rpy="-${pi/2} -${pi/2} -${pi/2} " xyz="0.085 0 0.088"/>
+   </joint>
+   <link name="plier_left">
+      <visual>
+         <origin xyz="0 0 0" />
+         <geometry>
+            <box size="0.02 0.15 0.15" />
+         </geometry>
+         <material name="">
+            <color rgba="0.79216 0.81961 0.93333 1" />
+         </material>
+      </visual>
+      <collision>
+         <origin xyz="0 0 0" />
+         <geometry>
+            <box size="0.02 0.15 0.15" />
+         </geometry>
+      </collision>
+      <xacro:inertial_box mass="0.5" x="0.02" y="0.15" z="0.15">
+         <origin xyz="0 0 0" rpy="0 0 0" />
+      </xacro:inertial_box>
+   </link>
+   <gazebo reference="plier_left">
+      <material>Gazebo/White</material>
+      <turnGravityOff>true</turnGravityOff>
+   </gazebo>
    <!-- TRANSMISSIONS -->
   <transmission name="arm_base_trans" type="SimpleTransmission">
